Commit message: yo

File: ARM_System/ROS/src_user/mastering_ros_robot/urdf/armstrong.xacro (robot description, xacro)
@@ -173,5 +173,5 @@
     <axis
       xyz="0 0 1" />
-    <limit lower="-3.14159265" upper="3.14159265" effort="24" velocity="6.07"/>
+    <limit lower="-1.5708" upper="1.5708" effort="24" velocity="6.07"/>
   </joint>
   <!-- //////////////////////////////////////////////////////////////////////////// -->
@@ -182,15 +182,15 @@
     <inertial>
       <origin
-        xyz="0.000201297618472596 0.00441389334559845 0.126754341902451"
-        rpy="0 0 0" />
-      <mass
-        value="0.205570337657311" />
-      <inertia
-        ixx="0.000945810095212874"
-        ixy="-3.75286422429002E-07"
-        ixz="-2.68834863919417E-06"
-        iyy="0.000980318138538167"
-        iyz="-8.22410793030225E-05"
-        izz="6.07849124063025E-05" />
+        xyz="0.000201293827647442 0.00441389267870827 0.12675435695043"
+        rpy="0 0 0" />
+      <mass
+        value="0.205570387117977" />
+      <inertia
+        ixx="0.000945810281839495"
+        ixy="-3.75279192756167E-07"
+        ixz="-2.68829797915708E-06"
+        iyy="0.000980318331283739"
+        iyz="-8.22410693097532E-05"
+        izz="6.07849054159079E-05" />
     </inertial>
     <visual>
@@ -279,5 +279,5 @@
     type="revolute">
     <origin
-      xyz="1.79999894011074E-05 0.0292119999936017 0.1917240000158"
+      xyz="1.79999894009408E-05 0.0292119999936017 0.1917240000158"
       rpy="3.32428011080213E-15 3.61394601646668E-15 -1.39659020047236E-14" />
     <parent
@@ -296,15 +296,15 @@
     <inertial>
       <origin
-        xyz="0.000275054818471177 -0.000920893443056015 0.0747617195797487"
-        rpy="0 0 0" />
-      <mass
-        value="0.127077319446387" />
-      <inertia
-        ixx="0.000160931457647102"
-        ixy="-3.20473054074497E-08"
-        ixz="-9.01217936692893E-07"
-        iyy="0.000160559888048535"
-        iyz="-5.01310156663423E-06"
-        izz="3.83030362883884E-07" />
+        xyz="0.000429978732766456 -7.0232266652509E-06 0.0337099670163837"
+        rpy="0 0 0" />
+      <mass
+        value="0.0812905905488399" />
+      <inertia
+        ixx="9.39737633066184E-06"
+        ixy="-1.04591568016406E-10"
+        ixz="-5.44323642033752E-08"
+        iyy="9.3976569237048E-06"
+        iyz="-1.8056954003407E-08"
+        izz="3.4998577136393E-10" />
     </inertial>
     <visual>
@@ -336,6 +336,6 @@
     type="revolute">
     <origin
-      xyz="0 -0.00674186407957562 0.1026461999984"
-      rpy="9.3132251030958E-21 0 1.3395654747779E-12" />
+      xyz="0 -0.00669799998980004 0.1003601999984"
+      rpy="-1.95701482895409E-16 -6.96589563095315E-15 2.30673060684073E-08" />
     <parent
       link="Link_4" />
@@ -393,6 +393,6 @@
     type="revolute">
     <origin
-      xyz="0 0 0.1179379999884"
-      rpy="-1.34193964960524E-12 -6.98884429251742E-09 -1.39659253553772E-14" />
+      xyz="0 0 0.0526599999884"
+      rpy="4.9973748652526E-07 -6.98884415650133E-09 -1.74585298068004E-14" />
     <parent
       link="Link_5" />
@@ -467,15 +467,15 @@
     <inertial>
       <origin
-        xyz="0.00860762646682772 0.00235992159407598 0.0393862951325977"
-        rpy="0 0 0" />
-      <mass
-        value="0.0270525603322218" />
-      <inertia
-        ixx="2.47548588580079E-05"
-        ixy="-8.63398014182299E-07"
-        ixz="6.42049429940404E-06"
-        iyy="2.66307768658301E-05"
-        iyz="1.05505702687199E-06"
-        izz="3.08245529576396E-06" />
+        xyz="0.0143 -0.023862 0.023722"
+        rpy="0 0 0" />
+      <mass
+        value="0.027053" />
+      <inertia
+        ixx="2.7531E-05"
+        ixy="-3.0411E-07"
+        ixz="-2.9977E-07"
+        iyy="2.9398E-06"
+        iyz="7.1644E-06"
+        izz="2.5394E-05" />
     </inertial>
     <visual>
@@ -507,6 +507,6 @@
     type="revolute">
     <origin
-      xyz="0.0186360000084232 -0.000852000011599824 0.041136000009572"
-      rpy="5.54546326711482E-17 1.39776847763541E-08 1.39659257005509E-14" />
+      xyz="0.0186360000084238 -0.000852000011599963 0.0411360000095722"
+      rpy="-1.17373567259265E-16 1.39776721927775E-08 -1.25987633750737E-16" />
     <parent
       link="Link_7" />
@@ -515,5 +515,5 @@
     <axis
       xyz="0 1 0" />
-    <limit lower="0" upper="1.00" effort="10" velocity="6.07"/>
+    <limit lower="0" upper="0.40" effort="10" velocity="6.07"/>
   </joint>
   <!-- //////////////////////////////////////////////////////////////////////////// -->
@@ -524,15 +524,15 @@
     <inertial>
       <origin
-        xyz="-0.00855603007043371 0.00235992159270827 0.0393975358112436"
-        rpy="0 0 0" />
-      <mass
-        value="0.0270525603322137" />
-      <inertia
-        ixx="2.47380022861504E-05"
-        ixy="8.64779209943437E-07"
-        ixz="-6.44885922745473E-06"
-        iyy="2.66307768658224E-05"
-        iyz="1.05392522348742E-06"
-        izz="3.09931186790004E-06" />
+        xyz="-0.014201 -0.024279 0.023724"
+        rpy="0 0 0" />
+      <mass
+        value="0.027053" />
+      <inertia
+        ixx="2.7501E-05"
+        ixy="3.9722E-07"
+        ixz="2.7586E-07"
+        iyy="2.935E-06"
+        iyz="7.1406E-06"
+        izz="2.5379E-05" />
     </inertial>
     <visual>
@@ -564,6 +564,6 @@
     type="revolute">
     <origin
-      xyz="-0.0186359999999997 -0.000852000011596368 0.041136"
-      rpy="-6.92750814262072E-15 1.39776987422794E-08 6.98296302286462E-15" />
+      xyz="-0.018636 -0.000426000011599953 0.0411359999999997"
+      rpy="-1.29121702479446E-16 1.39776998144446E-08 -1.24326241119813E-16" />
     <parent
       link="Link_7" />
@@ -572,5 +572,5 @@
     <axis
       xyz="0 1 0" />
-    <limit lower="-1.00" upper="0" effort="10" velocity="6.07"/>
+    <limit lower="-0.40" upper="0" effort="10" velocity="6.07"/>
     <mimic joint="Joint_7" multiplier="-1"/>
   </joint>
@@ -592,6 +592,6 @@
     type="fixed">
     <origin
-      xyz="2.12678282444645E-05 -0.00182300001159769 0.150049776923635"
-      rpy="3.54693587390868E-15 1.39776917593168E-08 6.98296302286467E-15" />
+      xyz="-2.40325633111271E-05 -0.0883617330439031 0.0805346693789171"
+      rpy="-4.99738824883467E-07 1.39776870622754E-08 -2.30659633733869E-08" />
     <parent
       link="Link_7" />

Commit message: 1_16_2019 - Changed code to be object oriented

File: ARM_System/ROS/src_user/mastering_ros_robot/urdf/armstrong.xacro (robot description, xacro)
@@ -24,17 +24,17 @@
   <link
     name="base_link">
-    <inertial>
-      <origin
-        xyz="-4.5737E-08 -0.020825 0.15228"
-        rpy="0 0 0" />
-      <mass
-        value="3.7701" />
-      <inertia
-        ixx="0.040053"
-        ixy="2.563E-08"
-        ixz="-5.9908E-08"
-        iyy="0.08344"
-        iyz="0.011411"
-        izz="0.052771" />
+		<inertial>
+      <origin
+        xyz="0.000642334886840512 -0.00918989728881375 0.15144445751703"
+        rpy="0 0 0" />
+      <mass
+        value="3.72304786520706" />
+      <inertia
+        ixx="0.0449452843063658"
+        ixy="-8.13830811365391E-05"
+        ixz="-0.000567018644234333"
+        iyy="0.0845135999112776"
+        iyz="-0.00256109565292216"
+        izz="0.0543313915567669" />
     </inertial>
     <visual>
